File: Hardware/VOLVOAUXBT.kicad_sch (KiCad schematic)
At the start: 66 parts, among them J1 Conn_01x01_Pin, J10 Conn_01x02_Pin, J11 Conn_01x02_Pin, J12 Conn_01x02_Pin, J13 Conn_01x05_Pin, J14 Conn_01x05_Pin, J15 Conn_01x02_Pin, J17 Conn_01x02_Pin, J18 Conn_01x05_Pin, J19 Conn_01x02_Pin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

Commit message: PCB layout wihtout traces
Parts:
- C1: renamed from C11; footprint (none) -> Capacitor_SMD:C_1206_3216Metric
- C10: renamed from C4; footprint (none) -> Capacitor_SMD:C_1206_3216Metric
- C11: renamed from C5; footprint (none) -> Capacitor_SMD:C_1206_3216Metric
- C12: renamed from C9; footprint (none) -> Capacitor_SMD:C_1206_3216Metric_Pad1.33x1.80mm_HandSolder
- C13: renamed from C8; footprint (none) -> Capacitor_SMD:C_1206_3216Metric_Pad1.33x1.80mm_HandSolder
- C14: renamed from C17; footprint (none) -> Capacitor_SMD:C_1206_3216Metric
- C15: renamed from C18; footprint (none) -> Capacitor_SMD:C_0805_2012Metric
- C16: renamed from C21; footprint (none) -> Capacitor_SMD:C_1206_3216Metric_Pad1.33x1.80mm_HandSolder
- C17: renamed from C3; footprint (none) -> Capacitor_SMD:C_1206_3216Metric
- C18: renamed from C22; footprint (none) -> Capacitor_SMD:C_1206_3216Metric_Pad1.33x1.80mm_HandSolder
- C19: renamed from C1; footprint (none) -> Capacitor_SMD:C_1206_3216Metric
- C2: renamed from C6; footprint (none) -> Capacitor_SMD:C_1206_3216Metric
- C20: footprint (none) -> Capacitor_SMD:C_0805_2012Metric
- C21: renamed from C19; footprint (none) -> Capacitor_SMD:C_0603_1608Metric
- C22: renamed from C2; footprint (none) -> Capacitor_SMD:C_1206_3216Metric
- C3: renamed from C7; footprint (none) -> Capacitor_SMD:C_1206_3216Metric
- C4: renamed from C12; footprint (none) -> Capacitor_SMD:C_1206_3216Metric
- C5: renamed from C13; footprint (none) -> Capacitor_SMD:C_1206_3216Metric
- C6: renamed from C14; footprint (none) -> Capacitor_SMD:C_1206_3216Metric
- C7: renamed from C15; footprint (none) -> Capacitor_SMD:C_1206_3216Metric
- C8: renamed from C16; footprint (none) -> Capacitor_SMD:C_1206_3216Metric
- C9: renamed from C10; footprint (none) -> Capacitor_SMD:C_1206_3216Metric_Pad1.33x1.80mm_HandSolder
- D1: footprint (none) -> Diode_SMD:D_1206_3216Metric
- J1: renamed from J9; footprint 10118193-0001LF:AMPHENOL_10118193-0001LF -> footprints3rd:AMPHENOL_10118193-0001LF
- J10: renamed from J11; footprint (none) -> Connector_PinHeader_2.54mm:PinHeader_1x02_P2.54mm_Vertical
- J11: renamed from J12; footprint (none) -> Connector_PinHeader_2.54mm:PinHeader_1x02_P2.54mm_Vertical
- J12: renamed from J13; footprint (none) -> Connector_PinHeader_2.54mm:PinHeader_1x05_P2.54mm_Vertical
- J13: renamed from J14; footprint (none) -> Connector_PinHeader_2.54mm:PinHeader_1x05_P2.54mm_Vertical
- J14: renamed from J18; footprint (none) -> Connector_JST:JST_XH_B5B-XH-AM_1x05_P2.50mm_Vertical
- J15: renamed from J19; footprint (none) -> Connector_PinHeader_2.54mm:PinHeader_1x02_P2.54mm_Vertical
- J16: renamed from J17; footprint (none) -> Connector_PinHeader_2.54mm:PinHeader_1x02_P2.54mm_Vertical
- J17: renamed from J1; footprint (none) -> Connector_PinHeader_2.54mm:PinHeader_1x01_P2.54mm_Vertical
- J18: renamed from J15; footprint (none) -> Connector_PinHeader_2.54mm:PinHeader_1x02_P2.54mm_Vertical
- J19: renamed from J7; footprint (none) -> Connector_PinHeader_2.54mm:PinHeader_1x01_P2.54mm_Vertical
- J2: renamed from J8; footprint 10118193-0001LF:AMPHENOL_10118193-0001LF -> footprints3rd:AMPHENOL_10118193-0001LF
- J3: renamed from J6; footprint F52R-1A7H1-11016:AMPHENOL_F52R-1A7H1-11016 -> footprints3rd:AMPHENOL_F52R-1A7H1-11018
- J4: renamed from J3; footprint (none) -> Connector_PinHeader_2.54mm:PinHeader_1x18_P2.54mm_Vertical
- J5: renamed from J4; footprint (none) -> Connector_PinHeader_2.54mm:PinHeader_1x18_P2.54mm_Vertical
- J6: renamed from J2; footprint F52R-1A7H1-11016:AMPHENOL_F52R-1A7H1-11016 -> footprints3rd:AMPHENOL_F52R-1A7H1-11018
- J7: renamed from J5; footprint (none) -> Connector_PinHeader_2.54mm:PinHeader_1x18_P2.54mm_Vertical
- J8: renamed from J20; footprint digikey-footprints:Coax_Conn_U.FL -> Connector_Coaxial:U.FL_Hirose_U.FL-R-SMT-1_Vertical
- J9: renamed from J10; footprint (none) -> Connector_PinHeader_2.54mm:PinHeader_1x02_P2.54mm_Vertical
- L1: footprint (none) -> Inductor_SMD:L_1206_3216Metric_Pad1.22x1.90mm_HandSolder
- R1: renamed from R18; footprint (none) -> Resistor_SMD:R_0603_1608Metric
- R10: renamed from R101; footprint (none) -> Resistor_SMD:R_0603_1608Metric
- R11: renamed from R1; footprint (none) -> Resistor_SMD:R_0603_1608Metric
- R12: renamed from R5; footprint (none) -> Resistor_SMD:R_0603_1608Metric
- R13: renamed from R3; footprint (none) -> Resistor_SMD:R_0603_1608Metric
- R14: renamed from R4; footprint (none) -> Resistor_SMD:R_0603_1608Metric
- R15: renamed from R2; footprint (none) -> Resistor_SMD:R_0603_1608Metric
- R2: renamed from R8; footprint (none) -> Resistor_SMD:R_0603_1608Metric
- R3: renamed from R6; footprint (none) -> Resistor_SMD:R_0603_1608Metric
- R4: renamed from R7; footprint (none) -> Resistor_SMD:R_0603_1608Metric
- R5: renamed from R106; footprint (none) -> Resistor_SMD:R_0603_1608Metric
- R6: renamed from R105; footprint (none) -> Resistor_SMD:R_0603_1608Metric
- R7: renamed from R104; footprint (none) -> Resistor_SMD:R_0603_1608Metric
- R8: renamed from R103; footprint (none) -> Resistor_SMD:R_0603_1608Metric
- R9: renamed from R102; footprint (none) -> Resistor_SMD:R_0603_1608Metric
- U1: renamed from U7; footprint Package_TO_SOT_SMD:TO-252-3_TabPin2 -> Package_TO_SOT_SMD:SOT-223-3_TabPin2
- U2: renamed from U9; footprint Package_TO_SOT_SMD:TO-252-3_TabPin2 -> Package_TO_SOT_SMD:SOT-223-3_TabPin2
- U3: renamed from U101; footprint TJA1027T_20_118:SOIC127P600X175-8N -> footprints3rd:SOIC127P600X175-8N
- U5: renamed from U102; footprint TJA1027T_20_118:SOIC127P600X175-8N -> footprints3rd:SOIC127P600X175-8N
- U6: renamed from U103; footprint SN74AHCT157PWR:SOP65P640X120-16N -> footprints3rd:SOP65P640X120-16N
- U7: renamed from U5; footprint Package_DFN_QFN:SiliconLabs_QFN-20-1EP_3x3mm_P0.5mm -> Package_DFN_QFN:SiliconLabs_QFN-20-1EP_3x3mm_P0.5mm_EP1.8x1.8mm_ThermalVias
- renumbered BTM2 to BTM1, U104 to U4
Connections:
- net BTM_GPIO_R3: no longer names the net of BTM1.6 (PIO15)
- no-connect marks 37 -> 38

Commit message: Before swap to wroom
Parts:
- added C23: 1uF/16V(10%), Capacitor_SMD:C_1206_3216Metric, symbol Device:C
- added C24: 10uF/25V(20%), Capacitor_SMD:C_1206_3216Metric, symbol Device:C
- added C25: 0.1uF/50V(10%), Capacitor_SMD:C_1206_3216Metric, symbol Device:C
- added J20, J21: Conn_01x05_Pin, Connector_PinHeader_2.54mm:PinHeader_1x05_P2.54mm_Vertical, symbol Connector:Conn_01x05_Pin
- added R16: 10K(1%), Resistor_SMD:R_0603_1608Metric, symbol Device:R
- added R17, R18, R19, R20, R21, R22, R23, R24: 500, Resistor_SMD:R_0603_1608Metric, symbol Device:R
- added U8: ESP32-WROOM-E, PCM_Espressif:ESP32-WROOM-32E, symbol PCM_Espressif:ESP32-WROOM-E
Connections:
- net BTM_GPIO_R1: now also R18.1
- net BTM_GPIO_R2: now also R17.1
- net BTM_NEXT: now also R20.1
- net BTM_ON/OFF: now also R24.1
- net BTM_PLAY: now also R19.1
- net BTM_PREVIOUS: now also R21.1
- net BTM_VOL+: now also R22.1
- net BTM_VOL-: now also R23.1
- net GND: now also C23.2, C24.2, C25.2, U8.1 (GND), U8.15 (GND), U8.38 (GND), U8.39 (GND_THERMAL)
- net GPIO0: now also U8.25 (GPIO0/BOOT/ADC2_CH1)
- net LIN1_RXD: now also U8.11 (DAC_2/ADC2_CH9/GPIO26)
- net LIN1_SLP: now also U8.9 (32K_XN/GPIO33/ADC1_CH5)
- net LIN1_TXD: now also U8.12 (ADC2_CH7/GPIO27)
- net LIN2_RXD: now also U8.28 (GPIO17)
- net LIN2_SLP: now also U8.8 (32K_XP/GPIO32/ADC1_CH4)
- net LIN2_TXD: now also U8.27 (GPIO16)
- net MB_CLK: now also J20.4 (Pin_4)
- net MB_D-MTS: now also J20.5 (Pin_5)
- net MB_D-STM: now also J20.3 (Pin_3)
- net MB_MTS: now also J20.2 (Pin_2)
- net MB_STM: now also J20.1 (Pin_1)
- net MUX_CONT: now also U8.26 (ADC2_CH0/GPIO4)
- net U0RXD: now also U8.34 (U0RXD/GPIO3)
- net U0TXD: now also U8.35 (U0TXD/GPIO1)
- net VCC_3V3: now also C24.1, C25.1, R16.1, U8.2 (3V3)
- new net: R23.2, U8.33 (GPIO21)
- new net: R21.2, U8.30 (GPIO18)
- new net: R22.2, U8.31 (GPIO19)
- new net: R24.2, U8.36 (GPIO22)
- new net: J21.5 (Pin_5), R18.2, U8.13 (MTMS/GPIO14/ADC2_CH6)
- new net: J21.1 (Pin_1), U8.5 (SENSOR_VN/GPIO39/ADC1_CH3)
- new net: J21.2 (Pin_2), U8.4 (SENSOR_VP/GPIO36/ADC1_CH0)
- new net: J21.3 (Pin_3), U8.7 (GPIO35/ADC1_CH7)
- new net: J21.4 (Pin_4), U8.6 (GPIO34/ADC1_CH6)
- new net: R20.2, U8.10 (DAC_1/ADC2_CH8/GPIO25)
- new net: C23.1, R16.2, U8.3 (EN/CHIP_PU)
- new net: R19.2, U8.37 (GPIO23)
- new net: R17.2, U8.16 (MTCK/GPIO13/ADC2_CH4)
- no-connect marks 38 -> 42
